File: fluidnc_board/spindle_cntrl.kicad_sch (KiCad schematic)
At the start: 63 parts

Commit message: remove unnecessary i2s chip
Other:
- title: (none) -> Spindle Control
Changed lines of the file:
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@@
 (kicad_sch (version 20211123) (generator eeschema)
   (paper "A4")
+  (title_block
+    (title "Spindle Control")
+  )
   (junction (at 140.335 98.425) (diameter 0) (color 0 0 0 0)
   )
