File: fluidnc_board/motor_drivers.kicad_sch (KiCad schematic)
At the start: 0 parts

Commit message: esp32 and motor driver stuff
Parts:
- added C? (x2): 100n, symbol Device:C
- added D?: B360, Diode_SMD:D_SMA_Handsoldering, symbol Diode:B360
- added U?: ADG3304, Package_SO:TSSOP-14_4.4x5mm_P0.65mm, symbol fluidnc_board:ADG3304
Connections:
- new net +3V3: C?.2, U?.1 (VCCA), U?.8 (EN)
- new net +48V: D?.1 (K)
- new net +5V: C?.1, D?.2 (A), U?.14 (VCCY)
- new net GND: C?.1, C?.2, U?.7 (GND)
- new net MISO: U?.3 (A2)
- new net MISO_5V: U?.12 (Y2)
- new net MOSI: U?.2 (A1)
- new net MOSI_5V: U?.13 (Y1)
- new net SCK: U?.4 (A3)
- new net SCK_5V: U?.11 (Y3)
- no-connect marks 0 -> 2
Other:
- added sheet driver_e (driver.kicad_sch)
- added sheet driver_y (driver.kicad_sch)
- added sheet driver_z (driver.kicad_sch)
- sheet driver_x: file driver_x.kicad_sch -> driver.kicad_sch
- sheet driver_x ports: added CS, DIR, EN, MISO, MOSI, SCK, STEP, VIO, VM; removed none

Commit message: remove unnecessary i2s chip
Other:
- title: (none) -> Motor Axes
Changed lines of the file:
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@@
 (kicad_sch (version 20211123) (generator eeschema)
   (paper "A4")
+  (title_block
+    (title "Motor Axes")
+  )
   (junction (at 149.225 109.22) (diameter 0) (color 0 0 0 0)
   )

Commit message: footprint associations and part no.
Parts:
- added C3: 100n, Capacitor_SMD:C_0603_1608Metric_Pad1.05x0.95mm_HandSolder, symbol Device:C
- added PS1: RKZ-2405S, fluidnc_board:CONV_RKZ, symbol fluidnc_board:RKZ-2405S
- C1, C2: renamed from C?; footprint (none) -> Capacitor_SMD:C_0603_1608Metric_Pad1.05x0.95mm_HandSolder; Digikey Part No. (none) -> 1276-1941-1-ND
- U1: renamed from U?; Digikey Part No. (none) -> 505-ADG3304BRUZ-ND
- gave numbers to parts that had none: 1
Connections:
- net +5V: now also PS1.1 (+VIN)
- net GND: now also PS1.2 (-VIN)
- new net 5V_ISO+: C3.1, PS1.7 (+VOUT)
- new net 5V_ISO-: C3.2, PS1.5 (-VOUT)
Other:
- sheet driver_e ports: added 5V_ISO, GND_ISO; removed none
- sheet driver_x ports: added 5V_ISO, GND_ISO; removed none
- sheet driver_y ports: added 5V_ISO, GND_ISO; removed none
- sheet driver_z ports: added 5V_ISO, GND_ISO; removed none

Commit message: fixed some footprint associations, placed footprints
Parts:
- C1, C2, C3: footprint Capacitor_SMD:C_0603_1608Metric_Pad1.05x0.95mm_HandSolder -> Capacitor_SMD:C_0603_1608Metric_Pad1.08x0.95mm_HandSolder; Digikey Part No. 1276-1941-1-ND -> (none)
- D1: Digikey Part No. CD214A-B360RCT-ND -> (none)
- PS1: Digikey Part No. 945-2566-ND -> (none); MANUFACTURER RECOM -> (none); MAXIMUM_PACKAGE_HEIGHT 10.2mm -> (none); PARTREV 5 -> (none); STANDARD Manufacturer Recommendations -> (none)
- U1: Digikey Part No. 505-ADG3304BRUZ-ND -> (none)
Changed lines of the file:
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@@
-      (effects (font (size 1.27 1.27)) hide)
-    )
-    (property "Digikey Part No." "505-ADG3304BRUZ-ND" (id 4) (at 161.29 128.27 0)
       (effects (font (size 1.27 1.27)) hide)
     )
@@
     (property "Reference" "C2" (id 0) (at 170.815 101.6 90))
     (property "Value" "100n" (id 1) (at 170.815 104.14 90))
-    (property "Footprint" "Capacitor_SMD:C_0603_1608Metric_Pad1.05x0.95mm_HandSolder" (id 2) (at 174.625 108.2548 0)
-      (effects (font (size 1.27 1.27)) hide)
-    )
-    (property "Datasheet" "http://www.samsungsem.com/kr/support/product-search/mlcc/CL10B104MB8NNNC.jsp" (id 3) (at 170.815 109.22 0)
-      (effects (font (size 1.27 1.27)) hide)
-    )
-    (property "Digikey Part No." "1276-1941-1-ND" (id 4) (at 170.815 109.22 0)
+    (property "Footprint" "Capacitor_SMD:C_0603_1608Metric_Pad1.08x0.95mm_HandSolder" (id 2) (at 174.625 108.2548 0)
+      (effects (font (size 1.27 1.27)) hide)
+    )
+    (property "Datasheet" "~" (id 3) (at 170.815 109.22 0)
       (effects (font (size 1.27 1.27)) hide)
     )
@@
       (effects (font (size 1.27 1.27)) hide)
     )
-    (property "Digikey Part No." "CD214A-B360RCT-ND" (id 4) (at 85.09 129.54 0)
-      (effects (font (size 1.27 1.27)) hide)
-    )
     (pin "1")
     (pin "2")
@@
     (property "Reference" "C1" (id 0) (at 143.51 101.6 90))
     (property "Value" "100n" (id 1) (at 143.51 104.14 90))
-    (property "Footprint" "Capacitor_SMD:C_0603_1608Metric_Pad1.05x0.95mm_HandSolder" (id 2) (at 147.32 108.2548 0)
-      (effects (font (size 1.27 1.27)) hide)
-    )
-    (property "Datasheet" "http://www.samsungsem.com/kr/support/product-search/mlcc/CL10B104MB8NNNC.jsp" (id 3) (at 143.51 109.22 0)
-      (effects (font (size 1.27 1.27)) hide)
-    )
-    (property "Digikey Part No." "1276-1941-1-ND" (id 4) (at 143.51 109.22 0)
+    (property "Footprint" "Capacitor_SMD:C_0603_1608Metric_Pad1.08x0.95mm_HandSolder" (id 2) (at 147.32 108.2548 0)
+      (effects (font (size 1.27 1.27)) hide)
+    )
+    (property "Datasheet" "~" (id 3) (at 143.51 109.22 0)
       (effects (font (size 1.27 1.27)) hide)
     )
@@
       (effects (font (size 1.27 1.27)) (justify left))
     )
-    (property "Footprint" "Capacitor_SMD:C_0603_1608Metric_Pad1.05x0.95mm_HandSolder" (id 2) (at 249.8852 129.54 0)
-      (effects (font (size 1.27 1.27)) hide)
-    )
-    (property "Datasheet" "http://www.samsungsem.com/kr/support/product-search/mlcc/CL10B104MB8NNNC.jsp" (id 3) (at 248.92 125.73 0)
-      (effects (font (size 1.27 1.27)) hide)
-    )
-    (property "Digikey Part No." "1276-1941-1-ND" (id 4) (at 248.92 125.73 0)
+    (property "Footprint" "Capacitor_SMD:C_0603_1608Metric_Pad1.08x0.95mm_HandSolder" (id 2) (at 249.8852 129.54 0)
+      (effects (font (size 1.27 1.27)) hide)
+    )
+    (property "Datasheet" "~" (id 3) (at 248.92 125.73 0)
       (effects (font (size 1.27 1.27)) hide)
     )
@@
       (effects (font (size 1.27 1.27)) (justify left bottom) hide)
     )
-    (property "Datasheet" "https://recom-power.com/pdf/Econoline/RKZ.pdf" (id 3) (at 229.235 125.73 0)
+    (property "Datasheet" "" (id 3) (at 229.235 125.73 0)
       (effects (font (size 1.27 1.27)) (justify left bottom) hide)
     )
-    (property "MAXIMUM_PACKAGE_HEIGHT" "10.2mm" (id 4) (at 229.235 125.73 0)
-      (effects (font (size 1.27 1.27)) (justify left bottom) hide)
-    )
-    (property "STANDARD" "Manufacturer Recommendations" (id 5) (at 229.235 125.73 0)
-      (effects (font (size 1.27 1.27)) (justify left bottom) hide)
-    )
-    (property "PARTREV" "5" (id 6) (at 229.235 125.73 0)
-      (effects (font (size 1.27 1.27)) (justify left bottom) hide)
-    )
-    (property "MANUFACTURER" "RECOM" (id 7) (at 229.235 125.73 0)
-      (effects (font (size 1.27 1.27)) (justify left bottom) hide)
-    )
-    (property "Digikey Part No." "945-2566-ND" (id 8) (at 229.235 125.73 0)
-      (effects (font (size 1.27 1.27)) hide)
-    )
-    (pin "1")
+    (pin "1")
