File: fluidnc_board/fluidnc_board.kicad_pcb (KiCad board)
At the start: 4 copper layers, 404 parts, among them J1 Conn_01x05_Female, J10 Screw_Terminal_01x04, J11 Screw_Terminal_01x02, J12 Conn_01x06_Female, J13 SWD, J14 Screw_Terminal_01x04, J15 Screw_Terminal_01x02, J16 Conn_01x06_Female, J17 SWD, J18 Screw_Terminal_01x04, J19 USB_B, J2 Micro_SD_Card_Det, J20 Screw_Terminal_01x04, J21 Screw_Terminal_01x02, J22 Screw_Terminal_01x03, J23 Screw_Terminal_01x06, J24 Screw_Terminal_01x03, J25 Screw_Terminal_01x03, J26 Screw_Terminal_01x03, J27 Screw_Terminal_01x03, J28 Screw_Terminal_01x02, J29 Screw_Terminal_01x02, J3 Screw_Terminal_01x02, J30 Screw_Terminal_01x02, J31 Screw_Terminal_01x02, J32 Screw_Terminal_01x02, J33 Screw_Terminal_01x02, J34 Screw_Terminal_01x02, J4 Conn_01x06_Female, J5 SWD, J6 Screw_Terminal_01x04, J7 Screw_Terminal_01x02, J8 Conn_01x06_Female, J9 SWD, Q1 IRF7809AVTRPBF, Q10 IRF9Z24SPBF, Q11 IRF7809AVTRPBF, Q12 IRF7809AVTRPBF, Q13 IRF7809AVTRPBF, Q14 IRF7809AVTRPBF, Q2 IRF7809AVTRPBF, Q3 IRF7809AVTRPBF, Q4 IRF7809AVTRPBF, Q5 SS8050-G, Q6 SS8050-G, Q7 BSS127S, Q8 BSS127S, Q9 ZVN4306GTA, SW1 SW_Push, SW2 SW_Push, SW3 SW_Push, SW4 SW_Push, SW5 SW_Push, SW6 SW_Push, U1 ADG3304, U10 ADG3304, U11 HCPL-0630, U12 STM32F103C8Tx, U13 TMC5160_SILENTSTEPSTICK, U14 ADG3304, U15 HCPL-0630, U16 STM32F103C8Tx, U17 TMC5160_SILENTSTEPSTICK, U18 CP2102N-Axx-xQFN28, U19 ESP32-WROOM-32UE, U2 ADG3304, U20 74HCT595, U21 74HCT595, U22 74HCT595, U23 BD9G341EFJ, U24 BD9G341EFJ, U25 BD9G341EFJ, U26 AZ1117-3.3, U27 HCPL-0630, U28 HCPL-0630, U29 HCPL-0630, U3 HCPL-0630, U30 HCPL-0630, U31 HCPL-0630, U32 HCPL-0630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

Commit message: placed and routed one stepper motor unit
Parts:
- removed C10, C11, C12, C13, C30, C31, C32, C36, C37, C38, C39, C4, C43, C44, C45, C49, C5, C50, C51, C52, C6: 100n, Capacitor_SMD:C_0603_1608Metric_Pad1.08x0.95mm_HandSolder
- removed C14, C40, C53: 47u, Capacitor_SMD:C_0805_2012Metric_Pad1.18x1.45mm_HandSolder
- removed C15, C41, C54: 4.7u, Capacitor_SMD:C_0805_2012Metric_Pad1.18x1.45mm_HandSolder
- removed C16, C42, C55: 100u, Capacitor_SMD:CP_Elec_10x10
- removed C33, C34, C46, C47, C7, C8: 22p, Capacitor_SMD:C_0603_1608Metric_Pad1.08x0.95mm_HandSolder
- removed C35, C48, C9: 12p, Capacitor_SMD:C_0402_1005Metric_Pad0.74x0.62mm_HandSolder
- removed D10, D11, D24, D25, D26, D27, D28, D29, D30, D31, D34, D35, D36, D37, D38, D39, D4, D40, D41, D5, D6, D7, D8, D9: B360, Diode_SMD:D_SMC
- removed D2, D22, D32: BZX84C5V6, Diode_SMD:D_SOT-23_ANK
- removed D23, D3, D33: LED, LED_SMD:LED_1206_3216Metric_Pad1.42x1.75mm_HandSolder
- removed J11, J15, J3: Screw_Terminal_01x02, Connector_Phoenix_MC:PhoenixContact_MC_1,5_2-G-3.81_1x02_P3.81mm_Horizontal
- removed J12, J16, J4: Conn_01x06_Female, Connector_JST:JST_XH_B6B-XH-A_1x06_P2.50mm_Vertical
- removed J13, J17, J5: SWD, Connector_PinHeader_2.54mm:PinHeader_1x05_P2.54mm_Vertical
- removed JP1, JP10, JP7: SolderJumper_3_Open, Jumper:SolderJumper-3_P1.3mm_Open_RoundedPad1.0x1.5mm_NumberLabels
- removed JP11, JP12, JP2, JP3, JP8, JP9: SolderJumper_3_Bridged12, Jumper:SolderJumper-3_P1.3mm_Bridged12_RoundedPad1.0x1.5mm_NumberLabels
- removed Q1, Q3, Q4: IRF7809AVTRPBF, Package_SO:SO-8_3.9x4.9mm_P1.27mm
- removed R10, R11, R28, R29, R37, R38: 100k, Resistor_SMD:R_0603_1608Metric_Pad0.98x0.95mm_HandSolder
- removed R21, R22, R3, R30, R31, R4: 270, Resistor_SMD:R_1206_3216Metric_Pad1.30x1.75mm_HandSolder
- removed R23, R27, R32, R36, R5, R9: 10k, Resistor_SMD:R_0805_2012Metric_Pad1.20x1.40mm_HandSolder
- removed R24, R25, R33, R34, R6, R7: 1k, Resistor_SMD:R_1206_3216Metric_Pad1.30x1.75mm_HandSolder
- removed R26, R35, R8: 100, Resistor_SMD:R_1206_3216Metric_Pad1.30x1.75mm_HandSolder
- removed SW1, SW3, SW4: SW_Push, Button_Switch_SMD:SW_Push_1P1T_NO_6x6mm_H9.5mm
- removed U10, U14, U2: ADG3304, Package_SO:TSSOP-14_4.4x5mm_P0.65mm
- removed U11, U15, U3: HCPL-0630, Package_SO:SOIC-8_3.9x4.9mm_P1.27mm
- removed U12, U16, U4: STM32F103C8Tx, Package_QFP:LQFP-48_7x7mm_P0.5mm
- removed U13, U17, U5: TMC5160_SILENTSTEPSTICK, fluidnc_board:TMC5160_SILENTSTEPSTICK
- removed Y1, Y3, Y4: 8M, Crystal:Crystal_SMD_3225-4Pin_3.2x2.5mm_HandSoldering
- C17, C18, C19, C20, C21, C23, C24, C25, C26, C27, D12, D13, D14, D16, D18, D20, Q2, R12, R13, R14, R15, R18, R19, R20, U6, U7, U8, Y2: moved to B.Cu
- C84: value 100n -> 100u; footprint Capacitor_SMD:C_0603_1608Metric_Pad1.08x0.95mm_HandSolder -> Capacitor_SMD:CP_Elec_10x10
- D1: footprint Diode_SMD:D_SMC -> Diode_SMD:D_SMA_Handsoldering
- D15, D17, D19, D21: moved to F.Cu
- R16: renamed from R17; moved to B.Cu
- R17: renamed from R16; moved to B.Cu
- RN1: footprint Package_SO:TSSOP-8_3x3mm_P0.65mm -> Package_SO:MSOP-8-1EP_3x3mm_P0.65mm_EP1.68x1.88mm_ThermalVias
- U23, U24, U25, U34: value BD9G341EFJ -> BD9G341AEFJ
- moved HS1 356.9 mm to (305.0, 407.1), turned to 0 degrees
- moved C87 160.7 mm to (-43.2, 78.7)
- moved C84 157.2 mm to (-43.2, 83.8)
- moved C88 155.5 mm to (-29.2, 78.7)
- moved U26 153.7 mm to (-36.8, 81.3)
- moved D51 111.6 mm to (-3.63, 101.2)
- moved F2 111.6 mm to (-3.68, 104.5)
- moved R71 111.6 mm to (-30.3, 130.4)
- moved C72 111.6 mm to (-54.6, 161.3)
- moved C76 111.6 mm to (-22.0, 103.1)
- moved C79 111.6 mm to (-80.2, 139.5)
- moved C80 111.6 mm to (-20.4, 127.3)
- moved C81 111.6 mm to (-52.3, 100.2)
- moved C83 111.6 mm to (-25.2, 130.6)
- moved C85 111.6 mm to (-18.8, 103.1)
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Connections:
- C91 pad 2: /spindle_cntrl/GND_VFD -> GND
- C92 pad 2: /spindle_cntrl/GND_VFD -> GND
- C93 pad 2: /spindle_cntrl/GND_VFD -> GND
- C94 pad 2: /spindle_cntrl/GND_VFD -> GND
- C95 pad 2: /spindle_cntrl/GND_VFD -> GND
- C98 pad 2: /spindle_cntrl/GND_VFD -> GND
- C99 pad 2: /spindle_cntrl/GND_VFD -> GND
- D52 pad 2: /spindle_cntrl/GND_VFD -> GND
- D53 pad 2: /spindle_cntrl/GND_VFD -> GND
- D54 pad 2: /spindle_cntrl/GND_VFD -> GND
- D56 pad 2: /spindle_cntrl/GND_VFD -> GND
- D57 pad 1: /spindle_cntrl/GND_VFD -> GND
- J28 pad 1: /spindle_cntrl/GND_VFD -> GND
- J30 pad 1: /spindle_cntrl/GND_VFD -> GND
- Q7 pad 2: /spindle_cntrl/GND_VFD -> GND
- Q8 pad 2: /spindle_cntrl/GND_VFD -> GND
- R101 pad 2: /spindle_cntrl/GND_VFD -> GND
- R104 pad 2: /spindle_cntrl/GND_VFD -> GND
- R106 pad 2: /spindle_cntrl/GND_VFD -> GND
- R108 pad 2: /spindle_cntrl/GND_VFD -> GND
- R94 pad 2: /spindle_cntrl/GND_VFD -> GND
- R99 pad 2: /spindle_cntrl/GND_VFD -> GND
- RN1 pad 2: /spindle_cntrl/GND_VFD -> GND
- RN1 pad 3: (no net) -> unconnected-(RN1-Pad3)
- RN1 pad 4: (no net) -> unconnected-(RN1-Pad4)
- RN1 pad 5: (no net) -> unconnected-(RN1-Pad5)
- RN1 pad 6: (no net) -> unconnected-(RN1-Pad6)
- U23 pad 9: (no net) -> GND
- U24 pad 9: (no net) -> GND
- U25 pad 9: (no net) -> GND
- U32 pad 5: /spindle_cntrl/GND_VFD -> GND
- U33 pad 5: /spindle_cntrl/GND_VFD -> GND
- U34 pad 2: /spindle_cntrl/GND_VFD -> GND
- U34 pad 9: (no net) -> GND
- U35 pad 4: /spindle_cntrl/GND_VFD -> GND
- U35 pad 5: Net-(C98-Pad1) -> Net-(R107-Pad1)
- U35 pad 6: Net-(R107-Pad2) -> Net-(R108-Pad1)
- U35 pad 7: Net-(R107-Pad2) -> Net-(R110-Pad1)
- U36 pad 1: (no net) -> unconnected-(U36-Pad1)
- U36 pad 2: (no net) -> unconnected-(U36-Pad2)
- U36 pad 3: (no net) -> unconnected-(U36-Pad3)
- U36 pad 4: /spindle_cntrl/GND_VFD -> GND
- U36 pad 5: Net-(R107-Pad1) -> Net-(C98-Pad1)
- U36 pad 6: Net-(R108-Pad1) -> Net-(R107-Pad2)
- U36 pad 7: Net-(R110-Pad1) -> Net-(R107-Pad2)
- U37 pad 4: /spindle_cntrl/GND_VFD -> GND
- U8 pad 39: /motor_drivers/driver_y/ENC_A -> unconnected-(U8-Pad39)
- U8 pad 40: /motor_drivers/driver_y/ENC_B -> unconnected-(U8-Pad40)
- U8 pad 41: unconnected-(U8-Pad41) -> /motor_drivers/driver_y/ENC_A
- U8 pad 42: unconnected-(U8-Pad42) -> /motor_drivers/driver_y/ENC_B
- U9 pad 11: Net-(D14-Pad2) -> Net-(D20-Pad2)
- U9 pad 12: Net-(D16-Pad2) -> Net-(D18-Pad2)
- U9 pad 13: Net-(D18-Pad2) -> Net-(D16-Pad2)
- U9 pad 14: Net-(D20-Pad2) -> Net-(D14-Pad2)
Routing:
- net GND: track 209.0 -> 58.9 mm, vias 0 -> 1
- net Net-(D20-Pad2): track 0.00 -> 127.3 mm
- net Net-(D16-Pad2): track 0.00 -> 121.3 mm
- net Net-(D18-Pad2): track 0.00 -> 100.9 mm
- net Net-(D14-Pad2): track 0.00 -> 95.8 mm
- net +3V3: track 153.8 -> 84.5 mm, vias 0 -> 3
- net /motor_drivers/driver_z/NRST: track 55.5 -> 0.00 mm
- net /motor_drivers/driver_e/NRST: track 55.5 -> 0.00 mm
- net /motor_drivers/driver_y/ENC_A: track 6.03 -> 34.7 mm, vias 2 -> 0
- net /motor_drivers/driver_x/NRST: track 25.4 -> 0.00 mm
- net /motor_drivers/driver_z/SWCLK: track 24.3 -> 0.00 mm, vias 1 -> 0
- net /motor_drivers/driver_e/SWCLK: track 24.3 -> 0.00 mm, vias 1 -> 0
- net /motor_drivers/driver_y/SWCLK: track 24.3 -> 0.00 mm, vias 1 -> 0
- net /motor_drivers/driver_y/ENC_B: track 2.95 -> 25.6 mm
- net Net-(J12-Pad4): track 22.5 -> 0.00 mm
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
Commit message: one driver unit layout
Parts:
- removed the C72 at (-54.6, 161.3)
- removed the C82 at (33.2, 162.2)
- removed the C83 at (-25.2, 130.6)
- removed the C84 at (-43.2, 83.8)
- removed the C85 at (-18.8, 103.1)
- removed the C86 at (-7.88, 113.2)
- removed the C87 at (-43.2, 78.7)
- removed the C88 at (-29.2, 78.7)
- removed the C89 at (-4.25, 107.7)
- removed the D49 at (-4.82, 97.2)
- removed the D50 at (-12.1, 110.3)
- removed the D51 at (-3.63, 101.2)
- removed the L3 at (33.2, 150.6)
- removed the R61 at (-48.7, 155.1)
- removed the R62 at (-34.1, 141.8)
- removed the R63 at (-38.4, 141.8)
- removed the R64 at (-20.3, 124.5)
- removed the R65 at (-25.0, 127.8)
- removed the R66 at (-46.0, 150.3)
- removed the R67 at (-6.94, 110.4)
- removed the R68 at (-13.0, 113.6)
- removed the R69 at (-25.7, 124.7)
- removed the R70 at (-53.8, 155.4)
- removed the R71 at (-30.3, 130.4)
- removed the U24 at (-10.9, 105.3)
- removed the U25 at (-52.6, 150.6)
- removed the U26 at (-36.8, 81.3)
- added C10: 100n, Capacitor_SMD:C_0603_1608Metric_Pad1.08x0.95mm_HandSolder, F.Cu at (476.2, 171.9)
- added C100: 6.8n, Capacitor_SMD:C_0402_1005Metric_Pad0.74x0.62mm_HandSolder, F.Cu at (-16.9, 14.6)
- added C101: 100n, Capacitor_SMD:C_0603_1608Metric_Pad1.08x0.95mm_HandSolder, F.Cu at (2.39, 114.4)
- added C11: 100n, Capacitor_SMD:C_0603_1608Metric_Pad1.08x0.95mm_HandSolder, F.Cu at (468.0, 159.5)
- added C12: 100n, Capacitor_SMD:C_0603_1608Metric_Pad1.08x0.95mm_HandSolder, F.Cu at (487.0, 162.0)
- added C13: 100n, Capacitor_SMD:C_0603_1608Metric_Pad1.08x0.95mm_HandSolder, F.Cu at (487.0, 159.5)
- added C14: 47u, Capacitor_SMD:C_0805_2012Metric_Pad1.18x1.45mm_HandSolder, F.Cu at (490.0, 155.3)
- added C15: 4.7u, Capacitor_SMD:C_0805_2012Metric_Pad1.18x1.45mm_HandSolder, F.Cu at (470.4, 174.4)
- added C16: 100u, Capacitor_SMD:CP_Elec_10x10, F.Cu at (447.8, 156.4)
- added C30: 100n, Capacitor_SMD:C_0603_1608Metric_Pad1.08x0.95mm_HandSolder, F.Cu at (337.4, 193.7)
- added C31: 100n, Capacitor_SMD:C_0603_1608Metric_Pad1.08x0.95mm_HandSolder, F.Cu at (382.4, 180.6)
- added C32: 100n, Capacitor_SMD:C_0603_1608Metric_Pad1.08x0.95mm_HandSolder, F.Cu at (396.0, 166.4)
- added C33: 22p, Capacitor_SMD:C_0603_1608Metric_Pad1.08x0.95mm_HandSolder, F.Cu at (400.3, 166.4)
- added C34: 22p, Capacitor_SMD:C_0603_1608Metric_Pad1.08x0.95mm_HandSolder, F.Cu at (397.9, 168.9)
- added C35: 12p, Capacitor_SMD:C_0402_1005Metric_Pad0.74x0.62mm_HandSolder, F.Cu at (364.2, 163.3)
- added C36: 100n, Capacitor_SMD:C_0603_1608Metric_Pad1.08x0.95mm_HandSolder, F.Cu at (393.6, 171.9)
- added C37: 100n, Capacitor_SMD:C_0603_1608Metric_Pad1.08x0.95mm_HandSolder, F.Cu at (385.4, 159.5)
- added C38: 100n, Capacitor_SMD:C_0603_1608Metric_Pad1.08x0.95mm_HandSolder, F.Cu at (404.4, 162.0)
- added C39: 100n, Capacitor_SMD:C_0603_1608Metric_Pad1.08x0.95mm_HandSolder, F.Cu at (404.4, 159.5)
- added C4: 100n, Capacitor_SMD:C_0603_1608Metric_Pad1.08x0.95mm_HandSolder, F.Cu at (420.0, 193.7)
- added C40: 47u, Capacitor_SMD:C_0805_2012Metric_Pad1.18x1.45mm_HandSolder, F.Cu at (407.4, 155.3)
- added C41: 4.7u, Capacitor_SMD:C_0805_2012Metric_Pad1.18x1.45mm_HandSolder, F.Cu at (387.8, 174.4)
- added C42: 100u, Capacitor_SMD:CP_Elec_10x10, F.Cu at (365.2, 156.4)
- added C43: 100n, Capacitor_SMD:C_0603_1608Metric_Pad1.08x0.95mm_HandSolder, F.Cu at (337.4, 241.4)
- added C44: 100n, Capacitor_SMD:C_0603_1608Metric_Pad1.08x0.95mm_HandSolder, F.Cu at (382.4, 228.4)
- added C45: 100n, Capacitor_SMD:C_0603_1608Metric_Pad1.08x0.95mm_HandSolder, F.Cu at (396.0, 214.1)
- added C46: 22p, Capacitor_SMD:C_0603_1608Metric_Pad1.08x0.95mm_HandSolder, F.Cu at (400.3, 214.1)
- added C47: 22p, Capacitor_SMD:C_0603_1608Metric_Pad1.08x0.95mm_HandSolder, F.Cu at (397.9, 216.6)
- added C48: 12p, Capacitor_SMD:C_0402_1005Metric_Pad0.74x0.62mm_HandSolder, F.Cu at (364.2, 211.1)
- added C49: 100n, Capacitor_SMD:C_0603_1608Metric_Pad1.08x0.95mm_HandSolder, F.Cu at (393.6, 219.6)
- added C5: 100n, Capacitor_SMD:C_0603_1608Metric_Pad1.08x0.95mm_HandSolder, F.Cu at (465.0, 180.6)
- added C50: 100n, Capacitor_SMD:C_0603_1608Metric_Pad1.08x0.95mm_HandSolder, F.Cu at (385.4, 207.3)
- added C51: 100n, Capacitor_SMD:C_0603_1608Metric_Pad1.08x0.95mm_HandSolder, F.Cu at (404.4, 209.8)
- added C52: 100n, Capacitor_SMD:C_0603_1608Metric_Pad1.08x0.95mm_HandSolder, F.Cu at (404.4, 207.3)
- added C53: 47u, Capacitor_SMD:C_0805_2012Metric_Pad1.18x1.45mm_HandSolder, F.Cu at (407.4, 203.1)
- added C54: 4.7u, Capacitor_SMD:C_0805_2012Metric_Pad1.18x1.45mm_HandSolder, F.Cu at (387.8, 222.2)
- added C55: 100u, Capacitor_SMD:CP_Elec_10x10, F.Cu at (365.2, 204.2)
- added C6: 100n, Capacitor_SMD:C_0603_1608Metric_Pad1.08x0.95mm_HandSolder, F.Cu at (478.6, 166.4)
- added C7: 22p, Capacitor_SMD:C_0603_1608Metric_Pad1.08x0.95mm_HandSolder, F.Cu at (482.9, 166.4)
- added C74: 100n, Capacitor_SMD:C_0603_1608Metric_Pad1.08x0.95mm_HandSolder, F.Cu at (-3.46, 95.3)
- added C76: 4.7u, Capacitor_SMD:C_0805_2012Metric_Pad1.18x1.45mm_HandSolder, F.Cu at (-25.4, 28.8)
- added C77: 100u, Capacitor_SMD:CP_Elec_10x10, F.Cu at (-22.9, 96.7)
- added C78: 4.7u, Capacitor_SMD:C_0805_2012Metric_Pad1.18x1.45mm_HandSolder, F.Cu at (-15.9, 107.5)
- added C8: 22p, Capacitor_SMD:C_0603_1608Metric_Pad1.08x0.95mm_HandSolder, F.Cu at (480.5, 168.9)
- added C9: 12p, Capacitor_SMD:C_0402_1005Metric_Pad0.74x0.62mm_HandSolder, F.Cu at (446.8, 163.3)
- added C96: 100n, Capacitor_SMD:C_0603_1608Metric_Pad1.08x0.95mm_HandSolder, F.Cu at (-35.2, 115.3)
- added C98: 100n, Capacitor_SMD:C_0603_1608Metric_Pad1.08x0.95mm_HandSolder, F.Cu at (-33.1, 88.0)
- added C99: 100n, Capacitor_SMD:C_0603_1608Metric_Pad1.08x0.95mm_HandSolder, F.Cu at (7.21, 115.9)
- added D10: B360, Diode_SMD:D_SMC, F.Cu at (443.0, 181.4)
- added D11: B360, Diode_SMD:D_SMC, F.Cu at (465.0, 165.7)
- added D2: BZX84C5V6, Diode_SMD:D_SOT-23_ANK, F.Cu at (459.4, 188.7)
- added D22: BZX84C5V6, Diode_SMD:D_SOT-23_ANK, F.Cu at (376.8, 188.7)
- added D23: LED, LED_SMD:LED_1206_3216Metric_Pad1.42x1.75mm_HandSolder, F.Cu at (390.9, 166.4)
- added D24: B360, Diode_SMD:D_SMC, F.Cu at (351.7, 189.1)
- added D25: B360, Diode_SMD:D_SMC, F.Cu at (399.5, 154.4)
- added D26: B360, Diode_SMD:D_SMC, F.Cu at (371.6, 174.0)
- added D27: B360, Diode_SMD:D_SMC, F.Cu at (388.7, 154.4)
- added D28: B360, Diode_SMD:D_SMC, F.Cu at (362.5, 189.1)
- added D29: B360, Diode_SMD:D_SMC, F.Cu at (371.6, 166.2)
- added D3: LED, LED_SMD:LED_1206_3216Metric_Pad1.42x1.75mm_HandSolder, F.Cu at (473.5, 166.4)
- added D30: B360, Diode_SMD:D_SMC, F.Cu at (360.4, 181.4)
- added D31: B360, Diode_SMD:D_SMC, F.Cu at (382.4, 165.7)
- added D32: BZX84C5V6, Diode_SMD:D_SOT-23_ANK, F.Cu at (376.8, 236.5)
- added D33: LED, LED_SMD:LED_1206_3216Metric_Pad1.42x1.75mm_HandSolder, F.Cu at (390.9, 214.2)
- added D34: B360, Diode_SMD:D_SMC, F.Cu at (351.7, 236.9)
- added D35: B360, Diode_SMD:D_SMC, F.Cu at (399.5, 202.2)
- added D36: B360, Diode_SMD:D_SMC, F.Cu at (371.6, 221.8)
- added D37: B360, Diode_SMD:D_SMC, F.Cu at (388.7, 202.2)
- added D38: B360, Diode_SMD:D_SMC, F.Cu at (362.5, 236.9)
- added D39: B360, Diode_SMD:D_SMC, F.Cu at (371.6, 214.0)
- added D4: B360, Diode_SMD:D_SMC, F.Cu at (434.3, 189.1)
- added D40: B360, Diode_SMD:D_SMC, F.Cu at (360.4, 229.1)
- added D41: B360, Diode_SMD:D_SMC, F.Cu at (382.4, 213.5)
- added D47: LED, LED_SMD:LED_1206_3216Metric_Pad1.42x1.75mm_HandSolder, F.Cu at (-16.2, 104.3)
- added D5: B360, Diode_SMD:D_SMC, F.Cu at (482.1, 154.4)
- added D6: B360, Diode_SMD:D_SMC, F.Cu at (454.2, 174.0)
- added D60: SS2150-LTP, Diode_SMD:D_SMA_Handsoldering, F.Cu at (-75.8, 24.3)
- added D61: SS2150-LTP, Diode_SMD:D_SMA_Handsoldering, F.Cu at (-28.4, 21.5)
- added D7: B360, Diode_SMD:D_SMC, F.Cu at (471.3, 154.4)
- added D8: B360, Diode_SMD:D_SMC, F.Cu at (445.1, 189.1)
- added D9: B360, Diode_SMD:D_SMC, F.Cu at (454.2, 166.2)
- added J11: Screw_Terminal_01x02, Connector_Phoenix_MC:PhoenixContact_MC_1,5_2-G-3.81_1x02_P3.81mm_Horizontal, F.Cu at (358.7, 168.5)
- added J12: Conn_01x06_Female, Connector_Molex:Molex_Micro-Fit_3.0_43045-0612_2x03_P3.00mm_Vertical, F.Cu at (338.7, 179.8)
- added J13: SWD, Connector_PinHeader_2.54mm:PinHeader_1x05_P2.54mm_Vertical, F.Cu at (355.5, 152.8)
- added J15: Screw_Terminal_01x02, Connector_Phoenix_MC:PhoenixContact_MC_1,5_2-G-3.81_1x02_P3.81mm_Horizontal, F.Cu at (358.7, 216.2)
- added J16: Conn_01x06_Female, Connector_Molex:Molex_Micro-Fit_3.0_43045-0612_2x03_P3.00mm_Vertical, F.Cu at (338.7, 227.5)
- added J17: SWD, Connector_PinHeader_2.54mm:PinHeader_1x05_P2.54mm_Vertical, F.Cu at (355.5, 200.6)
- added J3: Screw_Terminal_01x02, Connector_Phoenix_MC:PhoenixContact_MC_1,5_2-G-3.81_1x02_P3.81mm_Horizontal, F.Cu at (441.3, 168.5)
- added J4: Conn_01x06_Female, Connector_Molex:Molex_Micro-Fit_3.0_43045-0612_2x03_P3.00mm_Vertical, F.Cu at (421.3, 179.8)
- added J5: SWD, Connector_PinHeader_2.54mm:PinHeader_1x05_P2.54mm_Vertical, F.Cu at (438.1, 152.8)
- added JP1: SolderJumper_3_Open, Jumper:SolderJumper-3_P1.3mm_Open_RoundedPad1.0x1.5mm_NumberLabels, F.Cu at (460.0, 184.7)
- added JP10: SolderJumper_3_Open, Jumper:SolderJumper-3_P1.3mm_Open_RoundedPad1.0x1.5mm_NumberLabels, F.Cu at (377.4, 232.4)
- added JP11: SolderJumper_3_Bridged12, Jumper:SolderJumper-3_P1.3mm_Bridged12_RoundedPad1.0x1.5mm_NumberLabels, F.Cu at (377.4, 228.9)
- added JP12: SolderJumper_3_Bridged12, Jumper:SolderJumper-3_P1.3mm_Bridged12_RoundedPad1.0x1.5mm_NumberLabels, F.Cu at (399.1, 211.1)
- added JP2: SolderJumper_3_Bridged12, Jumper:SolderJumper-3_P1.3mm_Bridged12_RoundedPad1.0x1.5mm_NumberLabels, F.Cu at (460.0, 181.1)
- added JP3: SolderJumper_3_Bridged12, Jumper:SolderJumper-3_P1.3mm_Bridged12_RoundedPad1.0x1.5mm_NumberLabels, F.Cu at (481.7, 163.3)
- added JP7: SolderJumper_3_Open, Jumper:SolderJumper-3_P1.3mm_Open_RoundedPad1.0x1.5mm_NumberLabels, F.Cu at (377.4, 184.7)
- added JP8: SolderJumper_3_Bridged12, Jumper:SolderJumper-3_P1.3mm_Bridged12_RoundedPad1.0x1.5mm_NumberLabels, F.Cu at (377.4, 181.1)
- added JP9: SolderJumper_3_Bridged12, Jumper:SolderJumper-3_P1.3mm_Bridged12_RoundedPad1.0x1.5mm_NumberLabels, F.Cu at (399.1, 163.3)
- added L5: 33u, Inductor_SMD:L_Vishay_IHLP-4040, F.Cu at (-18.3, 26.0)
- added Q1: IRF7809AVTRPBF, Package_SO:SO-8_3.9x4.9mm_P1.27mm, F.Cu at (474.7, 161.5)
- added Q3: IRF7809AVTRPBF, Package_SO:SO-8_3.9x4.9mm_P1.27mm, F.Cu at (392.1, 161.5)
- added Q4: IRF7809AVTRPBF, Package_SO:SO-8_3.9x4.9mm_P1.27mm, F.Cu at (392.1, 209.3)
- added R10: 100k, Resistor_SMD:R_0603_1608Metric_Pad0.98x0.95mm_HandSolder, F.Cu at (476.2, 169.4)
- added R11: 100k, Resistor_SMD:R_0603_1608Metric_Pad0.98x0.95mm_HandSolder, F.Cu at (424.3, 193.7)
- added R112: 100k, Resistor_SMD:R_0603_1608Metric_Pad0.98x0.95mm_HandSolder, F.Cu at (-80.1, 17.8)
- added R113: 10k, Resistor_SMD:R_0805_2012Metric_Pad1.20x1.40mm_HandSolder, F.Cu at (-80.4, 19.7)
- added R116: 100k, Resistor_SMD:R_0603_1608Metric_Pad0.98x0.95mm_HandSolder, F.Cu at (-32.9, 15.0)
- added R117: 10k, Resistor_SMD:R_0805_2012Metric_Pad1.20x1.40mm_HandSolder, F.Cu at (-33.1, 16.9)
- added R118: 47k, Resistor_SMD:R_0805_2012Metric_Pad1.20x1.40mm_HandSolder, F.Cu at (-30.1, 12.3)
- added R119: 10k, Resistor_SMD:R_0805_2012Metric_Pad1.20x1.40mm_HandSolder, F.Cu at (-13.7, 14.7)
- added R21: 270, Resistor_SMD:R_1206_3216Metric_Pad1.30x1.75mm_HandSolder, F.Cu at (388.4, 171.3)
- added R22: 270, Resistor_SMD:R_1206_3216Metric_Pad1.30x1.75mm_HandSolder, F.Cu at (370.9, 191.7)
- added R23: 10k, Resistor_SMD:R_0805_2012Metric_Pad1.20x1.40mm_HandSolder, F.Cu at (360.2, 163.8)
- added R24: 1k, Resistor_SMD:R_1206_3216Metric_Pad1.30x1.75mm_HandSolder, F.Cu at (407.9, 152.2)
- added R25: 100, Resistor_SMD:R_1206_3216Metric_Pad1.30x1.75mm_HandSolder, F.Cu at (399.3, 159.9)
- added R26: 1k, Resistor_SMD:R_1206_3216Metric_Pad1.30x1.75mm_HandSolder, F.Cu at (380.0, 177.7)
- added R27: 10k, Resistor_SMD:R_0805_2012Metric_Pad1.20x1.40mm_HandSolder, F.Cu at (385.3, 177.5)
- added R28: 100k, Resistor_SMD:R_0603_1608Metric_Pad0.98x0.95mm_HandSolder, F.Cu at (393.6, 169.4)
- added R29: 100k, Resistor_SMD:R_0603_1608Metric_Pad0.98x0.95mm_HandSolder, F.Cu at (341.7, 193.7)
- added R3: 270, Resistor_SMD:R_1206_3216Metric_Pad1.30x1.75mm_HandSolder, F.Cu at (471.0, 171.3)
- added R30: 270, Resistor_SMD:R_1206_3216Metric_Pad1.30x1.75mm_HandSolder, F.Cu at (388.4, 219.0)
- added R31: 270, Resistor_SMD:R_1206_3216Metric_Pad1.30x1.75mm_HandSolder, F.Cu at (370.9, 239.5)
- added R32: 10k, Resistor_SMD:R_0805_2012Metric_Pad1.20x1.40mm_HandSolder, F.Cu at (360.2, 211.6)
- added R33: 1k, Resistor_SMD:R_1206_3216Metric_Pad1.30x1.75mm_HandSolder, F.Cu at (407.9, 199.9)
- added R34: 100, Resistor_SMD:R_1206_3216Metric_Pad1.30x1.75mm_HandSolder, F.Cu at (399.3, 207.7)
- added R35: 1k, Resistor_SMD:R_1206_3216Metric_Pad1.30x1.75mm_HandSolder, F.Cu at (380.0, 225.5)
- added R36: 10k, Resistor_SMD:R_0805_2012Metric_Pad1.20x1.40mm_HandSolder, F.Cu at (385.3, 225.3)
- added R37: 100k, Resistor_SMD:R_0603_1608Metric_Pad0.98x0.95mm_HandSolder, F.Cu at (393.6, 217.1)
- added R38: 100k, Resistor_SMD:R_0603_1608Metric_Pad0.98x0.95mm_HandSolder, F.Cu at (341.7, 241.4)
- added R4: 270, Resistor_SMD:R_1206_3216Metric_Pad1.30x1.75mm_HandSolder, F.Cu at (453.5, 191.7)
- added R5: 10k, Resistor_SMD:R_0805_2012Metric_Pad1.20x1.40mm_HandSolder, F.Cu at (442.8, 163.8)
- added R55: 12k, Resistor_SMD:R_0603_1608Metric_Pad0.98x0.95mm_HandSolder, F.Cu at (-63.8, 15.5)
- added R56: 270, Resistor_SMD:R_1206_3216Metric_Pad1.30x1.75mm_HandSolder, F.Cu at (-63.0, 13.5)
- added R57: 270, Resistor_SMD:R_1206_3216Metric_Pad1.30x1.75mm_HandSolder, F.Cu at (-57.9, 13.5)
- added R58: 270, Resistor_SMD:R_1206_3216Metric_Pad1.30x1.75mm_HandSolder, F.Cu at (-7.01, 92.4)
- added R59: 100, Resistor_SMD:R_1206_3216Metric_Pad1.30x1.75mm_HandSolder, F.Cu at (-1.06, 92.4)
- added R6: 1k, Resistor_SMD:R_1206_3216Metric_Pad1.30x1.75mm_HandSolder, F.Cu at (490.5, 152.2)
- added R7: 100, Resistor_SMD:R_1206_3216Metric_Pad1.30x1.75mm_HandSolder, F.Cu at (481.9, 159.9)
- added R8: 1k, Resistor_SMD:R_1206_3216Metric_Pad1.30x1.75mm_HandSolder, F.Cu at (462.6, 177.7)
- added R9: 10k, Resistor_SMD:R_0805_2012Metric_Pad1.20x1.40mm_HandSolder, F.Cu at (467.9, 177.5)
- added SW1: SW_Push, Button_Switch_SMD:SW_Push_1P1T_NO_6x6mm_H9.5mm, F.Cu at (423.3, 188.6)
- added SW3: SW_Push, Button_Switch_SMD:SW_Push_1P1T_NO_6x6mm_H9.5mm, F.Cu at (340.7, 188.6)
- added SW4: SW_Push, Button_Switch_SMD:SW_Push_1P1T_NO_6x6mm_H9.5mm, F.Cu at (340.7, 236.4)
- added U10: ADG3304, Package_SO:TSSOP-14_4.4x5mm_P0.65mm, F.Cu at (370.2, 181.1)
- added U11: HCPL-0630, Package_SO:SOIC-8_3.9x4.9mm_P1.27mm, F.Cu at (381.2, 172.8)
- added U12: STM32F103C8Tx, Package_QFP:LQFP-48_7x7mm_P0.5mm, F.Cu at (377.6, 156.2)
- added U13: TMC5160_SILENTSTEPSTICK, fluidnc_board:TMC5160_SILENTSTEPSTICK, F.Cu at (343.6, 165.3)
- added U14: ADG3304, Package_SO:TSSOP-14_4.4x5mm_P0.65mm, F.Cu at (370.2, 228.9)
- added U15: HCPL-0630, Package_SO:SOIC-8_3.9x4.9mm_P1.27mm, F.Cu at (381.2, 220.6)
- added U16: STM32F103C8Tx, Package_QFP:LQFP-48_7x7mm_P0.5mm, F.Cu at (377.6, 204.0)
- added U17: TMC5160_SILENTSTEPSTICK, fluidnc_board:TMC5160_SILENTSTEPSTICK, F.Cu at (343.6, 213.0)
- added U2: ADG3304, Package_SO:TSSOP-14_4.4x5mm_P0.65mm, F.Cu at (452.8, 181.1)
- added U23: AZ1117-3.3, Package_TO_SOT_SMD:SOT-89-3, F.Cu at (-13.1, 93.8)
- added U3: HCPL-0630, Package_SO:SOIC-8_3.9x4.9mm_P1.27mm, F.Cu at (463.8, 172.8)
- added U36: BD9G341AEFJ, Package_SO:HTSOP-8-1EP_3.9x4.9mm_P1.27mm_EP2.4x3.2mm_ThermalVias, F.Cu at (-72.4, 18.2)
- added U37: BD9G341AEFJ, Package_SO:HTSOP-8-1EP_3.9x4.9mm_P1.27mm_EP2.4x3.2mm_ThermalVias, F.Cu at (-25.0, 15.4)
- added U4: STM32F103C8Tx, Package_QFP:LQFP-48_7x7mm_P0.5mm, F.Cu at (460.2, 156.2)
- added U5: TMC5160_SILENTSTEPSTICK, fluidnc_board:TMC5160_SILENTSTEPSTICK, F.Cu at (426.2, 165.3)
- added Y1: 8M, Crystal:Crystal_SMD_3225-4Pin_3.2x2.5mm_HandSoldering, F.Cu at (453.9, 187.2)
- added Y3: 8M, Crystal:Crystal_SMD_3225-4Pin_3.2x2.5mm_HandSoldering, F.Cu at (371.3, 187.2)
- added Y4: 8M, Crystal:Crystal_SMD_3225-4Pin_3.2x2.5mm_HandSoldering, F.Cu at (371.3, 235.0)
- C80: value 100n -> 4.7u; footprint Capacitor_SMD:C_0603_1608Metric_Pad1.08x0.95mm_HandSolder -> Capacitor_SMD:C_0805_2012Metric_Pad1.18x1.45mm_HandSolder
- D48: value SS2150-LTP -> LED; footprint Diode_SMD:D_SMA_Handsoldering -> LED_SMD:LED_1206_3216Metric_Pad1.42x1.75mm_HandSolder
- J8: footprint Connector_JST:JST_XH_B6B-XH-A_1x06_P2.50mm_Vertical -> Connector_Molex:Molex_Micro-Fit_3.0_43045-0612_2x03_P3.00mm_Vertical
- R53: value 100k -> 3k
- R54: value 10k -> 750; footprint Resistor_SMD:R_0805_2012Metric_Pad1.20x1.40mm_HandSolder -> Resistor_SMD:R_0603_1608Metric_Pad0.98x0.95mm_HandSolder
- R82: renamed from R94; value 10k -> 2.2k; footprint Resistor_SMD:R_0805_2012Metric_Pad1.20x1.40mm_HandSolder -> Resistor_SMD:R_0603_1608Metric_Pad0.98x0.95mm_HandSolder
- moved HS1 321.2 mm to (361.7, 90.9), turned to 90 degrees
- moved U21 212.6 mm to (80.5, 128.8), turned to -90 degrees
- moved R108 208.7 mm to (-125.1, 33.0)
- moved R109 202.4 mm to (-125.3, 34.9), turned to 180 degrees
- moved R110 196.5 mm to (-120.6, 30.5), turned to 90 degrees
- moved R52 192.8 mm to (-106.9, 29.1)
- moved U35 189.0 mm to (-115.5, 33.6), turned to 180 degrees
- moved C71 188.0 mm to (-120.9, 23.7)
- moved R51 179.8 mm to (-106.9, 30.9), turned to 180 degrees
- moved C97 173.5 mm to (-64.3, 17.4)
- moved R114 167.7 mm to (-77.5, 15.1), turned to 90 degrees
- moved R115 165.0 mm to (-61.1, 17.5)
- moved U20 152.6 mm to (430.9, 201.6)
- moved U22 145.6 mm to (422.2, 201.6)
- moved R54 126.3 mm to (-16.4, 11.0)
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- renumbered C73 to C70, C74 to C72, C75 to C73, C81 to C75, C90 to C81, C91 to C82, C92 to C83, C93 to C84, C94 to C85, C95 to C86, C96 to C87, C97 to C88, C98 to C89, C99 to C90, C100 to C91, C101 to C92, C70 to C93, C76 to C94, C78 to C95, C77 to C97, D52 to D49, D53 to D50, D54 to D51, D55 to D52, D56 to D53, D57 to D54, D58 to D55, D59 to D56, D60 to D57, D61 to D58, D47 to D59, L5 to L2, L2 to L3, R112 to R100, R113 to R101, R114 to R102, R115 to R103, R116 to R104, R117 to R105, R118 to R106, R119 to R107, R51 to R108, R52 to R109, R55 to R110, R57 to R111, R56 to R114, R58 to R115, R59 to R51, R60 to R52, R72 to R60, R73 to R61, R74 to R62, R75 to R63, R76 to R64, R77 to R65, R78 to R66, R79 to R67, R80 to R68, R81 to R69, R82 to R70, R83 to R71, R84 to R72, R85 to R73, R86 to R74, R87 to R75, R88 to R76, R89 to R77, R90 to R78, R91 to R79, R92 to R80, R93 to R81, R95 to R83, R96 to R84, R97 to R85, R98 to R86, R99 to R87, R100 to R88, R101 to R89, R102 to R90, R103 to R91, R104 to R92, R105 to R93, R106 to R94, R107 to R95, R108 to R96, R109 to R97, R110 to R98, R111 to R99, U27 to U24, U28 to U25, U29 to U26, U30 to U27, U31 to U28, U32 to U29, U33 to U30, U34 to U31, U36 to U32, U35 to U33, U37 to U34, U23 to U35
Connections:
- net Net-(C81-Pad1) renamed /power_supply/regulator/OUT
- net Net-(R53-Pad2) renamed /power_supply/regulator2/FB
- net Net-(R59-Pad2) renamed /power_supply/regulator/FB
- C79 pad 1: Net-(C79-Pad1) -> +3V3
- C79 pad 2: Net-(C79-Pad2) -> GND
- C80 pad 1: +48V -> /power_supply/regulator1/OUT
- D48 pad 1: Net-(C79-Pad2) -> GND
- D48 pad 2: GND -> Net-(D48-Pad2)
- F2 pad 2: Net-(C82-Pad1) -> /power_supply/regulator2/OUT
- F3 pad 2: Net-(C89-Pad1) (its old number) -> /power_supply/regulator1/OUT
- J8 pad 3: Net-(J8-Pad3) -> Net-(U7-Pad4)
- J8 pad 4: Net-(J8-Pad4) -> Net-(R12-Pad2)
- J8 pad 5: Net-(J8-Pad5) -> Net-(U7-Pad2)
- L4 pad 2: Net-(C89-Pad1) (its old number) -> /power_supply/regulator1/OUT
- R12 pad 2: Net-(J8-Pad5) -> Net-(R12-Pad2)
- R13 pad 2: Net-(J8-Pad3) -> Net-(J8-Pad2)
- R53 pad 1: +48V -> /power_supply/regulator2/OUT
- U6 pad 10: /STEP_Y -> /DIR_Y
- U6 pad 11: /DIR_Y -> /STEP_Y
- U6 pad 4: /motor_drivers/driver_y/DIR_3V3 -> /motor_drivers/driver_y/STEP_3V3
- U6 pad 5: /motor_drivers/driver_y/STEP_3V3 -> /motor_drivers/driver_y/DIR_3V3
- U7 pad 2: Net-(J8-Pad4) -> Net-(U7-Pad2)
- U7 pad 4: Net-(J8-Pad2) -> Net-(U7-Pad4)
- U8 pad 27: /motor_drivers/driver_y/STEP_3V3 -> /motor_drivers/driver_y/DIR_3V3
- U8 pad 28: /motor_drivers/driver_y/DIR_3V3 -> /motor_drivers/driver_y/STEP_3V3
Routing:
- net Net-(U7-Pad4): track 0.00 -> 38.7 mm
- net /motor_drivers/driver_y/SWCLK: track 0.00 -> 36.3 mm, vias 0 -> 1
- net /power_supply/regulator1/OUT: track 0.00 -> 34.2 mm, vias 0 -> 2
- net Net-(U7-Pad2): track 0.00 -> 34.2 mm
- net /power_supply/regulator2/OUT: track 0.00 -> 32.8 mm, vias 0 -> 2
- net +3V3: track 84.5 -> 51.9 mm, vias 3 -> 2
- net /power_supply/regulator/OUT: track 0.00 -> 30.5 mm, vias 0 -> 2
- net Net-(R12-Pad2): track 0.00 -> 29.5 mm
- net /motor_drivers/driver_y/ENC_A: track 34.7 -> 5.48 mm
- net Net-(C70-Pad1): track 0.00 -> 26.2 mm
- net Net-(J8-Pad4): track 17.5 -> 0.00 mm
- net /motor_drivers/driver_y/ENC_B: track 25.6 -> 8.23 mm
- net /motor_drivers/driver_y/STEP_DRV: track 0.00 -> 17.1 mm
- net Net-(C95-Pad2): track 0.00 -> 15.4 mm
- net Net-(C101-Pad2): track 0.00 -> 15.4 mm
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